Commit message: Reverse j5 and j10 joint axis direction
- j5:  1 0 0 → -1 0 0
- j10: -1 0 0 → 1 0 0

Co-Authored-By: Claude Sonnet 4.6 <noreply@anthropic.com>

File: assets/dual_arm/urdf/dual_arm_assembly.urdf (robot description, URDF)
Before this commit: robot dual_arm_assembly, 11 links, 10 joints
Joints:
- joint j10: axis -1 0 0 -> 1 0 0
- joint j5: axis 1 0 0 -> -1 0 0
